File: f1c200s.kicad_pcb (KiCad board)
At the start: 2 copper layers, 62 x 46 mm, 58 parts, among them J1 Conn_02x14_Odd_Even, J10 Conn_02x04_Odd_Even, J11 105162-0001, J12 10118194-0011LF, J13 Conn_01x06_Male, J14 Conn_01x06_Male, J2 Conn_01x04_Male, J3 Conn_01x07_Male, J4 Conn_02x03_Odd_Even, J5 Conn_01x03_Male, J6 Conn_01x04_Male, J7 Conn_02x04_Odd_Even, J8 Conn_01x06_Male, J9 Conn_01x01_Male, SW1 SW_Push, U1 AP2127N-3.3, U2 F1C100s, U3 XC6421AB03ER-G, U4 AT25xxx, Y1 24MHz

Commit message: second rev of crap board
Parts:
- added C20: .1u, Capacitor_SMD:C_0603_1608Metric_Pad1.05x0.95mm_HandSolder, F.Cu at (227.3, 59.2)
- added C21: .1u, Capacitor_SMD:C_0603_1608Metric_Pad1.05x0.95mm_HandSolder, F.Cu at (224.4, 58.8)
- added C22: .1u, Capacitor_SMD:C_0603_1608Metric_Pad1.05x0.95mm_HandSolder, F.Cu at (222.8, 58.7)
- added J15: 105162-0001, 105162-0001:105162-0001, F.Cu at (229.7, 28.3)
- added R12: 220k, Capacitor_SMD:C_0603_1608Metric_Pad1.05x0.95mm_HandSolder, F.Cu at (220.3, 58.0)
- added R13: 220k, Capacitor_SMD:C_0603_1608Metric_Pad1.05x0.95mm_HandSolder, F.Cu at (220.3, 59.5)
- R10: value 2.2k -> 10k
- R11: value 3.3k -> 220k; footprint Resistor_SMD:R_0603_1608Metric_Pad1.05x0.95mm_HandSolder -> Capacitor_SMD:C_0603_1608Metric_Pad1.05x0.95mm_HandSolder
- U1: value AP2127N-3.3 -> 3.3v
- moved R11 49.1 mm to (229.1, 59.2), turned to 270 degrees
- moved U4 12.2 mm to (232.5, 35.6), turned to 90 degrees
- moved R10 11.8 mm to (264.6, 22.9), turned to 270 degrees
- moved J5 9.58 mm to (227.3, 61.9), turned to 270 degrees
- moved JP1 8.09 mm to (229.7, 35.6), turned to 270 degrees
- moved J11 6.61 mm to (222.4, 26.9), turned to 270 degrees
- moved JP4 6.41 mm to (225.2, 32.6), turned to 90 degrees
- moved J6 5.62 mm to (232.6, 29.9)
- moved JP2 5.33 mm to (239.3, 32.7), turned to 90 degrees
- moved JP3 5.31 mm to (236.8, 32.7), turned to 90 degrees
- moved R9 4.14 mm to (228.0, 32.8), turned to 180 degrees
- moved J13 3.90 mm to (227.0, 35.6)
- moved U1 0.07 mm to (249.5, 29.1), turned to 0 degrees
Connections:
- J4 pad 6: Net-(J4-Pad6) -> /COM
- J5 pad 1: /COM -> Net-(C20-Pad2)
- J5 pad 2: /L -> Net-(C21-Pad2)
- J5 pad 3: /R -> Net-(C22-Pad2)
- JP6 pad 1: Net-(JP6-Pad1) -> Net-(J12-Pad4)
- R10 pad 1: Net-(J12-Pad4) -> +3V3
- R10 pad 2: Net-(JP6-Pad1) -> Net-(J12-Pad4)
- R11 pad 1: Net-(JP6-Pad1) -> /MIC
- U1 pad 1: GND -> +3V3
- U1 pad 2: +3V3 -> +5V
- U1 pad 3: +5V -> GND
- U2 pad 86: Net-(J4-Pad6) -> Net-(J4-Pad5)
- U2 pad 87: Net-(J4-Pad5) -> /MIC
Routing:
- net /SPI_0_CS: track 19.8 -> 46.8 mm
- net /SPI_0_CLK: track 16.5 -> 35.2 mm
- net /SPI_0_MISO: track 18.0 -> 33.7 mm, vias 1 -> 2
- net Net-(J4-Pad6): track 14.6 -> 0.00 mm
- net /SPI_0_MOSI: track 19.6 -> 32.4 mm, vias 2 -> 1
- net /D-: track 57.9 -> 69.9 mm
- net /D+: track 59.5 -> 71.4 mm
- net /MIC: track 0.00 -> 11.2 mm, vias 0 -> 2
- net +3V3: track 228.9 -> 239.8 mm, vias 2 -> 5
- net /COM: track 22.2 -> 32.5 mm
- net /SDC0_CLK: track 28.5 -> 37.5 mm
- net /SDC0_D0: track 30.7 -> 39.4 mm
- net /SDC0_D2: track 23.0 -> 31.5 mm
- net /SDC0_CMD: track 26.2 -> 34.5 mm
- net /SDC0_D3: track 24.6 -> 32.8 mm
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